Commit message: Add localizer package back in and add base-link in properly (#15)
* added dependencies script and requirements.txt

* add localizer package back in and add base-link in properly

just rename chassis base link no need for new link

* added geographic lib to dependencies.sh

* add parameters and proper imu and gps transforms for localizer

* add ground truth odometry

* fix world loading and sensors

* removed test package, added node functionality, renamed to just localizer

* make more realistic

* remove old .rviz file

File: src/description/urdf/athena_drive.urdf.xacro (robot description, xacro)
@@ -11,4 +11,5 @@
   <xacro:include filename="imu.xacro"/>
   <xacro:include filename="gps.xacro"/>
+  <xacro:include filename="ground_truth_odom.xacro"/>
   <!-- Load robot's macro with parameters -->
   <!-- set prefix if multiple robots are used -->
@@ -26,4 +27,11 @@
   <!-- Contains description of drive -->
   <xacro:description/>
+  <xacro:imu_sensor parent="base_link">
+    <origin xyz="0 0 0.0" rpy="0 0 0"/>
+  </xacro:imu_sensor>
+  <xacro:gps_sensor parent="base_link">
+    <origin xyz="0 0 0.0" rpy="0 0 0"/>
+  </xacro:gps_sensor>
+  <xacro:ground_truth_odometry/>
   <xacro:if value="$(arg use_mock_hardware)">
     <xacro:athena_drive_ros2_control

File: src/description/urdf/athena_drive_description.urdf.xacro (robot description, xacro)
@@ -5,5 +5,5 @@
 <robot xmlns:xacro="http://www.ros.org/wiki/xacro">
     <xacro:macro name="description">
-        <link name="chassis_base_link">
+        <link name="base_link">
             <inertial>
                 <origin xyz="0.775305042176281 -0.0692748019047986 -0.475175318827691" rpy="0 0 0" />
@@ -51,5 +51,5 @@
         <joint name="suspension_front_left_joint" type="fixed">
             <origin xyz="0.61263 0.22146 -0.74592" rpy="1.5708 0 0.094743" />
-            <parent link="chassis_base_link" />
+            <parent link="base_link" />
             <child link="suspension_front_left_link" />
             <axis xyz="0 0 -1" />
@@ -306,5 +306,5 @@
         <joint name="suspension_front_right_joint" type="fixed">
             <origin xyz="0.66803 -0.36146 -0.74592" rpy="1.5708 0 0.094743" />
-            <parent link="chassis_base_link" />
+            <parent link="base_link" />
             <child link="suspension_front_right_link" />
             <axis xyz="0 0 1" />

File: src/description/urdf/gps.xacro (robot description, xacro)
@@ -1,11 +1,11 @@
 <?xml version="1.0"?>
 <robot xmlns:xacro="http://www.ros.org/wiki/xacro">
-    <xacro:macro name="gps_sensor" params="parent prefix *origin">
-        <joint name="${prefix}_gps_joint" type="fixed">
+    <xacro:macro name="gps_sensor" params="parent *origin">
+        <joint name="gnss_joint" type="fixed">
             <xacro:insert_block name="origin" />
             <parent link="${parent}" />
-            <child link="${prefix}_gps_link" />
+            <child link="gnss_link" />
         </joint>
-        <link name="${prefix}_gps_link">
+        <link name="gnss_link">
             <visual>
                 <geometry>
@@ -17,11 +17,11 @@
             </visual>
         </link>
-        <gazebo reference="${prefix}_gps_link">
-            <sensor name="${prefix}_navsat" type="navsat">
+        <gazebo reference="gnss_link">
+            <sensor name="navsat" type="navsat">
                 <always_on>true</always_on>
-                <update_rate>10</update_rate>
-                <topic>/gps</topic>
-                <plugin filename="libgz-sim-navsat-system.so" name="gz::sim::systems::NavSat">
-                </plugin>
+                <update_rate>50</update_rate>
+                <topic>/gps/fix</topic>
+                <ign_frame_id>gnss_link</ign_frame_id>
+                <plugin filename="ignition-gazebo-navsat-system" name="ignition::gazebo::systems::NavSat"/>
             </sensor>
         </gazebo>

File: src/description/urdf/imu.xacro (robot description, xacro)
@@ -1,11 +1,11 @@
 <?xml version="1.0"?>
 <robot xmlns:xacro="http://www.ros.org/wiki/xacro">
-    <xacro:macro name="imu_sensor" params="parent prefix *origin">
-        <joint name="${prefix}_imu_joint" type="fixed">
+    <xacro:macro name="imu_sensor" params="parent *origin">
+        <joint name="imu_joint" type="fixed">
             <xacro:insert_block name="origin" />
             <parent link="${parent}" />
-            <child link="${prefix}_imu_link" />
+            <child link="imu_link" />
         </joint>
-        <link name="${prefix}_imu_link">
+        <link name="imu_link">
             <visual>
                 <geometry>
@@ -17,10 +17,11 @@
             </visual>
         </link>
-        <gazebo reference="${prefix}_imu_link">
-            <sensor name="${prefix}_imu" type="imu">
+        <gazebo reference="imu_link">
+            <sensor name="imu" type="imu">
                 <always_on>true</always_on>
-                <update_rate>100</update_rate>
+                <update_rate>200</update_rate>
                 <topic>/imu</topic>
-                <plugin filename="libgz-sim-imu-system.so" name="gz::sim::systems::Imu"/>
+                <ign_frame_id>imu_link</ign_frame_id>
+                <plugin filename="libignition-gazebo-imu-system.so" name="ignition::gazebo::systems::Imu"/>
             </sensor>
         </gazebo>

Commit message: added depth camera to urdf

File: src/description/urdf/athena_drive.urdf.xacro (robot description, xacro)
@@ -12,4 +12,5 @@
   <xacro:include filename="gps.xacro"/>
   <xacro:include filename="ground_truth_odom.xacro"/>
+  <xacro:include filename="depth_camera.xacro"/>
   <!-- Load robot's macro with parameters -->
   <!-- set prefix if multiple robots are used -->
@@ -34,4 +35,7 @@
   </xacro:gps_sensor>
   <xacro:ground_truth_odometry/>
+  <xacro:depth_camera parent_link="base_link">
+      <origin xyz="0.75 0 -0.37" rpy="0 0 0"/>
+  </xacro:depth_camera>
   <xacro:if value="$(arg use_mock_hardware)">
     <xacro:athena_drive_ros2_control
